File: replicate_layout_test_project/replicate_layout_test_project.kicad_pcb (KiCad board)
At the start: 2 copper layers, 71 parts, among them J1001 Pusa_6mm, J1002 Pusa_6mm, J201 Pusa_6mm, J202 Pusa_6mm, J601 Pusa_6mm, J602 Pusa_6mm, Q1101 CSD19531KCS, Q1102 CSD19531KCS, Q1301 CSD19531KCS, Q1302 CSD19531KCS, Q1401 CSD19531KCS, Q1402 CSD19531KCS, Q301 CSD19531KCS, Q302 CSD19531KCS, Q501 CSD19531KCS, Q502 CSD19531KCS, Q701 CSD19531KCS, Q702 CSD19531KCS, Q901 CSD19531KCS, Q902 CSD19531KCS, U101 TMS320F28027DA, U1101 IR2181, U1201 INA240A1D, U1301 IR2181, U1401 IR2181, U301 IR2181, U401 INA240A1D, U501 IR2181, U701 IR2181, U801 INA240A1D, U901 IR2181

Commit message: updated test project
Parts:
- removed C301, C302, C501, C502: 1u, Passives:C1206M
- removed D1101, D1301, D1401, D301, D501, D701, D901: 1N4148, Diode_SMD:D_MiniMELF
- removed J1001, J1002, J201, J202, J601, J602: Pusa_6mm, Connector:Pusa_6mm
- removed Q1101, Q1102, Q1301, Q1302, Q1401, Q1402, Q301, Q302, Q501, Q502, Q701, Q702, Q901, Q902: CSD19531KCS, Discretes:TO-220
- removed R1501: R1206, Passives:R1206M
- removed R301, R302, R501, R502: 20R, Passives:R1206M
- removed the REF** at (82.5, 141.0)
- removed U301, U501: IR2181, Package_SO:SO8
- added C1001: C, Capacitor_SMD:C_1206_3216Metric, F.Cu at (227.1, 145.7)
- added C1002: C, Capacitor_SMD:C_1206_3216Metric, F.Cu at (227.1, 149.1)
- added C1003: C, Capacitor_SMD:C_1206_3216Metric, F.Cu at (227.1, 152.4)
- added C1004: C, Capacitor_SMD:C_1206_3216Metric, F.Cu at (214.4, 162.6)
- added C101: C, Capacitor_SMD:C_1206_3216Metric, F.Cu at (191.2, 115.3)
- added C102: C, Capacitor_SMD:C_1206_3216Metric, F.Cu at (191.2, 118.6)
- added C1103: C, Capacitor_SMD:C_1206_3216Metric, F.Cu at (245.1, 133.6)
- added C1104: C, Capacitor_SMD:C_1206_3216Metric, F.Cu at (214.4, 157.2)
- added C1201: C, Capacitor_SMD:C_1206_3216Metric, F.Cu at (209.2, 126.9)
- added C1202: C, Capacitor_SMD:C_1206_3216Metric, F.Cu at (209.2, 130.2)
- added C1203: C, Capacitor_SMD:C_1206_3216Metric, F.Cu at (209.2, 133.6)
- added C1204: C, Capacitor_SMD:C_1206_3216Metric, F.Cu at (214.4, 151.9)
- added C1303: C, Capacitor_SMD:C_1206_3216Metric, F.Cu at (245.1, 114.8)
- added C1304: C, Capacitor_SMD:C_1206_3216Metric, F.Cu at (206.8, 151.9)
- added C1403: C, Capacitor_SMD:C_1206_3216Metric, F.Cu at (191.2, 143.1)
- added C1404: C, Capacitor_SMD:C_1206_3216Metric, F.Cu at (199.1, 151.9)
- added C401: C, Capacitor_SMD:C_1206_3216Metric, F.Cu at (100.3, 63.3)
- added C402: C, Capacitor_SMD:C_1206_3216Metric, B.Cu at (111.1, 62.7)
- added C403: C, Capacitor_SMD:C_1206_3216Metric, F.Cu at (121.9, 64.6)
- added C404: C, Capacitor_SMD:C_1206_3216Metric, B.Cu at (109.9, 68.2)
- added C703: C, Capacitor_SMD:C_1206_3216Metric, F.Cu at (190.9, 82.0)
- added C704: C, Capacitor_SMD:C_1206_3216Metric, F.Cu at (189.2, 63.9)
- added C801: C, Capacitor_SMD:C_1206_3216Metric, F.Cu at (227.1, 108.1)
- added C802: C, Capacitor_SMD:C_1206_3216Metric, F.Cu at (227.1, 111.4)
- added C803: C, Capacitor_SMD:C_1206_3216Metric, F.Cu at (227.1, 114.8)
- added C804: C, Capacitor_SMD:C_1206_3216Metric, F.Cu at (199.1, 162.6)
- added C903: C, Capacitor_SMD:C_1206_3216Metric, F.Cu at (209.2, 114.8)
- added C904: C, Capacitor_SMD:C_1206_3216Metric, F.Cu at (199.1, 157.2)
- added J101: In, Connector_PinHeader_2.54mm:PinHeader_1x02_P2.54mm_Vertical, F.Cu at (190.7, 108.7)
- added J102: Out, Connector_PinHeader_2.54mm:PinHeader_1x02_P2.54mm_Vertical, F.Cu at (195.4, 108.7)
- added R1001: R, Resistor_SMD:R_1206_3216Metric, F.Cu at (221.5, 138.9)
- added R1002: R, Resistor_SMD:R_1206_3216Metric, F.Cu at (221.5, 142.2)
- added R1003: R, Resistor_SMD:R_1206_3216Metric, F.Cu at (221.5, 145.5)
- added R1004: R, Resistor_SMD:R_1206_3216Metric, F.Cu at (221.5, 148.8)
- added R101: R, Resistor_SMD:R_1206_3216Metric, F.Cu at (185.6, 101.3)
- added R102: R, Resistor_SMD:R_1206_3216Metric, F.Cu at (185.6, 104.5)
- added R103: R, Resistor_SMD:R_1206_3216Metric, F.Cu at (185.6, 107.8)
- added R104: R, Resistor_SMD:R_1206_3216Metric, F.Cu at (185.6, 111.1)
- added R105: R, Resistor_SMD:R_1206_3216Metric, F.Cu at (185.6, 114.4)
- added R106: R, Resistor_SMD:R_1206_3216Metric, F.Cu at (185.6, 117.7)
- added R107: R, Resistor_SMD:R_1206_3216Metric, F.Cu at (185.6, 121.0)
- added R108: R, Resistor_SMD:R_1206_3216Metric, F.Cu at (185.6, 124.3)
- added R1103: R, Resistor_SMD:R_1206_3216Metric, F.Cu at (239.5, 126.7)
- added R1104: R, Resistor_SMD:R_1206_3216Metric, F.Cu at (239.5, 129.9)
- added R1202: R, Resistor_SMD:R_1206_3216Metric, F.Cu at (203.5, 123.4)
- added R1203: R, Resistor_SMD:R_1206_3216Metric, F.Cu at (203.5, 126.7)
- added R1204: R, Resistor_SMD:R_1206_3216Metric, F.Cu at (203.5, 129.9)
- added R1303: R, Resistor_SMD:R_1206_3216Metric, F.Cu at (239.5, 107.8)
- added R1304: R, Resistor_SMD:R_1206_3216Metric, F.Cu at (239.5, 111.1)
- added R1403: R, Resistor_SMD:R_1206_3216Metric, F.Cu at (185.6, 136.2)
- added R1404: R, Resistor_SMD:R_1206_3216Metric, F.Cu at (185.6, 139.4)
- added R402: R, Resistor_SMD:R_1206_3216Metric, F.Cu at (103.5, 63.3)
- added R403: R, Resistor_SMD:R_1206_3216Metric, F.Cu at (110.7, 69.8)
- added R404: R, Resistor_SMD:R_1206_3216Metric, F.Cu at (118.7, 64.6)
- added R703: R, Resistor_SMD:R_1206_3216Metric, F.Cu at (185.2, 75.0)
- added R704: R, Resistor_SMD:R_1206_3216Metric, F.Cu at (185.2, 78.3)
- added R802: R, Resistor_SMD:R_1206_3216Metric, F.Cu at (221.5, 104.5)
- added R803: R, Resistor_SMD:R_1206_3216Metric, F.Cu at (221.5, 107.8)
- added R804: R, Resistor_SMD:R_1206_3216Metric, F.Cu at (221.5, 111.1)
- added R903: R, Resistor_SMD:R_1206_3216Metric, F.Cu at (203.5, 107.8)
- added R904: R, Resistor_SMD:R_1206_3216Metric, F.Cu at (203.5, 111.1)
- added REF**: KiCad-Logo_6mm_SilkScreen, Symbol:KiCad-Logo_6mm_SilkScreen, F.Cu at (189.2, 173.4)
- added U1001: NE5532, Package_SO:SOIC-8_5.23x5.23mm_P1.27mm, B.Cu at (110.5, 88.3)
- C1101, C1102, C1301, C1302, C1402, C701, C901, C902: value 1u -> C; footprint Passives:C1206M -> Capacitor_SMD:C_1206_3216Metric
- C1401, C702: value 1u -> C; footprint Passives:C1206M -> Capacitor_SMD:C_1206_3216Metric; moved to F.Cu
- R1101, R1102, R1301, R1302, R1401, R1402, R901, R902: value 20R -> R; footprint Passives:R1206M -> Resistor_SMD:R_1206_3216Metric
- R1201, R401, R801: value R_Shunt -> R; footprint Passives:RM -> Resistor_SMD:R_1206_3216Metric
- R701, R702: value 20R -> R; footprint Passives:R1206M -> Resistor_SMD:R_1206_3216Metric; moved to F.Cu
- U101: value TMS320F28027DA -> NE5532; footprint Package_SO:TSSOP-38_4.4x9.7mm_P0.5mm -> Package_SO:SOIC-8_5.23x5.23mm_P1.27mm
- U1101, U1301, U1401, U901: value IR2181 -> NE5532; footprint Package_SO:SO8 -> Package_SO:SOIC-8_5.23x5.23mm_P1.27mm
- U1201, U401, U801: value INA240A1D -> NE5532; footprint Package_SO:SOIC-8_3.9x4.9mm_P1.27mm -> Package_SO:SOIC-8_5.23x5.23mm_P1.27mm
- U701: value IR2181 -> NE5532; footprint Package_SO:SO8 -> Package_SO:SOIC-8_5.23x5.23mm_P1.27mm; moved to F.Cu
- moved U1401 182.5 mm to (61.2, 61.6), turned to 180 degrees
- moved U801 146.0 mm to (109.2, 43.2), turned to 20 degrees
- moved U101 99.5 mm to (193.6, 103.0)
- moved R1302 92.4 mm to (239.5, 104.5)
- moved C1301 91.8 mm to (245.1, 108.1)
- moved U1301 86.4 mm to (247.4, 103.0)
- moved R1301 81.6 mm to (239.5, 101.3)
- moved R1402 81.0 mm to (185.6, 132.9), turned to 0 degrees
- moved C1302 75.8 mm to (245.1, 111.4)
- moved C1402 74.2 mm to (191.2, 139.7), turned to 0 degrees
- moved C1401 74.2 mm to (191.2, 136.4), turned to 0 degrees
- moved R1401 67.2 mm to (185.6, 129.6), turned to 0 degrees
- moved R902 67.0 mm to (203.5, 104.5)
- moved C901 65.0 mm to (209.2, 108.1)
- moved C1101 62.7 mm to (245.1, 126.9)
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Connections:
- C1101 pad 1: +15V -> /Cascade2/low_pass1/mid
- C1101 pad 2: GND -> Net-(U1101A--)
- C1102 pad 1: /Full Bridge2/Leg+/VB -> +15V
- C1102 pad 2: /Full Bridge2/Leg+/VS -> GND
- C1301 pad 1: +15V -> /Cascade3/low_pass1/mid
- C1301 pad 2: GND -> Net-(U1301A--)
- C1302 pad 1: /Full Bridge2/Leg-/VB -> +15V
- C1302 pad 2: /Full Bridge2/Leg-/VS -> GND
- C1401 pad 1: +15V -> /low_pass2/mid
- C1401 pad 2: GND -> Net-(U1401A--)
- C1402 pad 1: /Leg+1/VB -> +15V
- C1402 pad 2: /Leg+1/VS -> GND
- C701 pad 1: +15V -> /Cascade/low_pass/mid
- C701 pad 2: GND -> Net-(U701A--)
- C702 pad 1: /Full Bridge1/Leg+/VB -> +15V
- C702 pad 2: /Full Bridge1/Leg+/VS -> GND
- C901 pad 1: +15V -> /Cascade1/low_pass1/mid
- C901 pad 2: GND -> Net-(U901A--)
- C902 pad 1: /Full Bridge1/Leg-/VB -> +15V
- C902 pad 2: /Full Bridge1/Leg-/VS -> GND
- R1101 pad 1: Net-(R1101-Pad1) -> /Cascade2/low_pass/out
- R1101 pad 2: Net-(Q1101-Pad1) -> Net-(U1101A--)
- R1102 pad 1: Net-(R1102-Pad1) -> Net-(U1101A--)
- R1102 pad 2: Net-(Q1102-Pad1) -> /Cascade2/low_pass1/mid
- R1201 pad 1: /Full Bridge2/Current sensor/OUT -> /Cascade/in
- R1201 pad 2: Net-(R1201-Pad2) -> Net-(U1201A--)
- R1301 pad 1: Net-(R1301-Pad1) -> /Cascade3/low_pass/out
- R1301 pad 2: Net-(Q1301-Pad1) -> Net-(U1301A--)
- R1302 pad 1: Net-(R1302-Pad1) -> Net-(U1301A--)
- R1302 pad 2: Net-(Q1302-Pad1) -> /Cascade3/low_pass1/mid
- R1401 pad 1: Net-(R1401-Pad1) -> /Cascade/in
- R1401 pad 2: Net-(Q1401-Pad1) -> Net-(U1401A--)
- R1402 pad 1: Net-(R1402-Pad1) -> Net-(U1401A--)
- R1402 pad 2: Net-(Q1402-Pad1) -> /low_pass2/mid
- R401 pad 1: /Full Bridge/Current sensor/OUT -> /Cascade/low_pass/out
- R401 pad 2: Net-(R401-Pad2) -> Net-(U401A--)
- R701 pad 1: Net-(R701-Pad1) -> /Cascade/in
- R701 pad 2: Net-(Q701-Pad1) -> Net-(U701A--)
- R702 pad 1: Net-(R702-Pad1) -> Net-(U701A--)
- R702 pad 2: Net-(Q702-Pad1) -> /Cascade/low_pass/mid
- R801 pad 1: /Full Bridge1/Current sensor/OUT -> /Cascade/in
- R801 pad 2: Net-(R801-Pad2) -> Net-(U801A--)
- R901 pad 1: Net-(R901-Pad1) -> /Cascade1/low_pass/out
- R901 pad 2: Net-(Q901-Pad1) -> Net-(U901A--)
- R902 pad 1: Net-(R902-Pad1) -> Net-(U901A--)
- R902 pad 2: Net-(Q902-Pad1) -> /Cascade1/low_pass1/mid
- U101 pad 1: unconnected-(U101-Pad1) -> Net-(R106-Pad2)
- U101 pad 2: GND -> Net-(U101A--)
- U101 pad 3: unconnected-(U101-Pad3) -> GND
- U101 pad 4: +3V3 -> -15V
- U101 pad 5: /Full Bridge1/Q_high -> GND
- U101 pad 6: /Full Bridge1/Q_low -> Net-(U101B--)
- U101 pad 7: /Full Bridge2/Q_high -> Net-(J102-Pin_1)
- U101 pad 8: /Full Bridge2/Q_low -> +15V
- U1101 pad 1: /Full Bridge2/Q_high -> /Cascade2/low_pass1/mid
- U1101 pad 2: /Full Bridge2/Q_low -> Net-(U1101A--)
- U1101 pad 4: Net-(R1102-Pad1) -> -15V
- U1101 pad 5: +15V -> GND
- U1101 pad 6: /Full Bridge2/Leg+/VS -> Net-(U1101B--)
- U1101 pad 7: Net-(R1101-Pad1) -> /Cascade2/out
- U1101 pad 8: /Full Bridge2/Leg+/VB -> +15V
- U1201 pad 1: Net-(R1201-Pad3) -> /Cascade3/low_pass/mid
- U1201 pad 2: GND -> Net-(U1201A--)
- U1201 pad 3: +3V3 -> GND
- U1201 pad 4: GND -> -15V
- U1201 pad 5: /Full Bridge2/current -> GND
- U1201 pad 6: +3V3 -> Net-(U1201B--)
- U1201 pad 7: GND -> /Cascade3/low_pass/out
- U1201 pad 8: Net-(R1201-Pad2) -> +15V
- U1301 pad 1: /Full Bridge2/Q_low -> /Cascade3/low_pass1/mid
- U1301 pad 2: /Full Bridge2/Q_high -> Net-(U1301A--)
- U1301 pad 4: Net-(R1302-Pad1) -> -15V
- U1301 pad 5: +15V -> GND
- U1301 pad 6: /Full Bridge2/Leg-/VS -> Net-(U1301B--)
- U1301 pad 7: Net-(R1301-Pad1) -> /Cascade3/out
- U1301 pad 8: /Full Bridge2/Leg-/VB -> +15V
- U1401 pad 1: /Leg+1/Q_HIGH -> /low_pass2/mid
- U1401 pad 2: /Leg+1/Q_LOW -> Net-(U1401A--)
- U1401 pad 4: Net-(R1402-Pad1) -> -15V
- U1401 pad 5: +15V -> GND
- U1401 pad 6: /Leg+1/VS -> Net-(U1401B--)
- U1401 pad 7: Net-(R1401-Pad1) -> /low_pass2/out
- U1401 pad 8: /Leg+1/VB -> +15V
- U401 pad 1: Net-(R401-Pad3) -> /Cascade/low_pass1/mid
- U401 pad 2: GND -> Net-(U401A--)
- U401 pad 3: +3V3 -> GND
- U401 pad 4: GND -> -15V
- U401 pad 5: /Full Bridge/current -> GND
- U401 pad 6: +3V3 -> Net-(U401B--)
- U401 pad 7: GND -> /Cascade/out
- U401 pad 8: Net-(R401-Pad2) -> +15V
- U701 pad 1: /Full Bridge1/Q_high -> /Cascade/low_pass/mid
- U701 pad 2: /Full Bridge1/Q_low -> Net-(U701A--)
- U701 pad 4: Net-(R702-Pad1) -> -15V
- U701 pad 5: +15V -> GND
- U701 pad 6: /Full Bridge1/Leg+/VS -> Net-(U701B--)
- U701 pad 7: Net-(R701-Pad1) -> /Cascade/low_pass/out
- U701 pad 8: /Full Bridge1/Leg+/VB -> +15V
- U801 pad 1: Net-(R801-Pad3) -> /Cascade1/low_pass/mid
- U801 pad 2: GND -> Net-(U801A--)
- U801 pad 3: +3V3 -> GND
- U801 pad 4: GND -> -15V
- U801 pad 5: /Full Bridge1/current -> GND
- U801 pad 6: +3V3 -> Net-(U801B--)
- U801 pad 7: GND -> /Cascade1/low_pass/out
- U801 pad 8: Net-(R801-Pad2) -> +15V
- U901 pad 1: /Full Bridge1/Q_low -> /Cascade1/low_pass1/mid
- U901 pad 2: /Full Bridge1/Q_high -> Net-(U901A--)
- U901 pad 4: Net-(R902-Pad1) -> -15V
- U901 pad 5: +15V -> GND
- U901 pad 6: /Full Bridge1/Leg-/VS -> Net-(U901B--)
- U901 pad 7: Net-(R901-Pad1) -> /Cascade1/out
- U901 pad 8: /Full Bridge1/Leg-/VB -> +15V
Routing:
- net /Leg+1/VS: track 59.1 -> 0.00 mm
- net +3V3: track 39.0 -> 0.00 mm
- net /Full Bridge/current: track 35.0 -> 0.00 mm
- net /Full Bridge/Leg-/VS: track 30.9 -> 0.00 mm
- net /Full Bridge/Leg+/VS: track 30.9 -> 0.00 mm, vias 1 -> 0
- net Net-(R1402-Pad1): track 27.4 -> 0.00 mm
- net GND: track 0.00 -> 21.0 mm, vias 0 -> 2
- net /Leg+1/VB: track 21.0 -> 0.00 mm, vias 2 -> 0
- net +VDC: track 20.3 -> 0.00 mm
- net /Full Bridge/Leg+/VB: track 16.5 -> 0.00 mm, vias 1 -> 0
- net Net-(R1401-Pad1): track 15.8 -> 0.00 mm
- net /Cascade/low_pass1/mid: track 0.00 -> 15.5 mm
- net /Leg+1/Q_HIGH: track 14.9 -> 0.00 mm
- net /Full Bridge/Q_low: track 14.3 -> 0.00 mm
- net /Full Bridge/Q_high: track 14.3 -> 0.00 mm
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- added copper zone on F.Cu, net -15V
- added copper zone on B.Cu, net GND
- removed copper zone on B.Cu, net /Full Bridge/Current sensor/OUT
- removed copper zone on F.Cu, net /Full Bridge/Current sensor/OUT
- removed copper zone on F.Cu, net /Full Bridge/Leg+/VS
- removed copper zone on F.Cu, net /Full Bridge/Leg-/VS
- removed copper zone on F.Cu, net /Leg+1/VS
Other:
- board text added: "K"
- board text removed: "B"
- board text removed: "Comment"
- board text removed: "group_locked"
- board text removed: "locked"

Commit message: update test project
Parts:
- added C1501: C, Capacitor_SMD:C_1206_3216Metric, B.Cu at (81.1, 86.6)
- added C1502: C, Capacitor_SMD:C_1206_3216Metric, F.Cu at (80.4, 97.4)
- added C1503: C, Capacitor_SMD:C_1206_3216Metric, F.Cu at (85.9, 96.1)
- added C1504: C, Capacitor_SMD:C_1206_3216Metric, B.Cu at (82.3, 108.2)
- added R109: R, Resistor_SMD:R_1206_3216Metric, F.Cu at (250.6, 142.7)
- added R1501: R, Resistor_SMD:R_1206_3216Metric, B.Cu at (82.5, 82.6)
- added R1502: R, Resistor_SMD:R_1206_3216Metric, B.Cu at (81.1, 89.8)
- added R1503: R, Resistor_SMD:R_1206_3216Metric, B.Cu at (87.6, 96.9)
- added R1504: R, Resistor_SMD:R_1206_3216Metric, B.Cu at (82.4, 105.0)
- added U1501: NE5532, Package_SO:SOIC-8_5.23x5.23mm_P1.27mm, B.Cu at (83.2, 96.9)
- C702, C704: moved to B.Cu
- moved C702 81.9 mm to (111.3, 58.9), turned to -90 degrees
- moved C704 79.1 mm to (110.1, 64.3), turned to -90 degrees
- moved R703 74.9 mm to (110.9, 66.0)
- moved C703 71.9 mm to (122.1, 60.8), turned to -90 degrees
- moved R704 68.6 mm to (119.0, 60.8), turned to 90 degrees
- moved U701 45.9 mm to (110.9, 61.6)
- moved R702 45.7 mm to (103.7, 59.5)
- moved C701 41.6 mm to (100.5, 59.5)
- moved R701 40.6 mm to (96.5, 61.0)
- moved C402 30.3 mm to (141.2, 58.9)
- moved R401 30.3 mm to (126.4, 61.0)
- moved R402 30.3 mm to (133.6, 59.5)
- moved R403 30.3 mm to (140.7, 66.0)
- moved R404 30.3 mm to (148.8, 60.8)
- moved C401 30.3 mm to (130.4, 59.5)
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Routing:
- net GND: track 21.0 -> 63.1 mm, vias 2 -> 6
- net /Cascade/low_pass/mid: track 0.00 -> 15.5 mm
- net /low_pass3/mid: track 0.00 -> 15.5 mm
- net Net-(U701B--): track 0.00 -> 13.1 mm
- net Net-(U1501B--): track 0.00 -> 13.1 mm
- net -15V: track 5.26 -> 15.8 mm, vias 1 -> 3
- net +15V: track 5.25 -> 15.7 mm, vias 1 -> 3
- net Net-(U701A--): track 0.00 -> 9.31 mm
- net Net-(U1501A--): track 0.00 -> 9.31 mm
- net /Cascade/low_pass/out: track 0.00 -> 8.32 mm
- net /low_pass3/out: track 0.00 -> 8.32 mm
- added copper zone on B.Cu, net -15V
- added copper zone on F.Cu, net GND
