File: replicate_layout_test_project/replicate_layout_test_project.kicad_pcb (KiCad board)
At the start: 2 copper layers, 105 parts, among them J101 In, J102 Out, U1001 NE5532, U101 NE5532, U1101 NE5532, U1201 NE5532, U1301 NE5532, U1401 NE5532, U1501 NE5532, U401 NE5532, U701 NE5532, U801 NE5532, U901 NE5532

Commit message: towards V10 compatible release
Parts:
- U801: moved to B.Cu
- moved U801 24.2 mm to (110.0, 19.0), turned to -20 degrees
