File: replicate_layout_test_project/low_pass.kicad_sch (KiCad schematic)
At the start: 9 parts, among them U401 NE5532

Commit message: towards V10 compatible release
Parts:
- renumbered C701 to C401, C703 to C403, R702 to R402, R703 to R403, R704 to R404
